Commit message: added gazebo control with gazebo hardware interface

File: description/camera.xacro (robot description, xacro)
@@ -4,5 +4,5 @@
         <parent link="chassis"/>
         <child link="camera_link"/>
-        <origin xyz="0.170 0 0" rpy="0 0 0"/>
+        <origin xyz="0.0425 0 0" rpy="0 0 0"/>
     </joint>
     <link name="camera_link">

File: description/lidar.xacro (robot description, xacro)
@@ -26,5 +26,5 @@
         <sensor name="laser" type="ray">
             <pose> 0 0 0 0 0 0 </pose>
-            <visualize>true</visualize>
+            <visualize>false</visualize>
             <update_rate>10</update_rate>
             <ray>

File: description/robot.urdf.xacro (robot description, xacro)
@@ -2,7 +2,7 @@
 <robot xmlns:xacro="http://www.ros.org/wiki/xacro"  name="robot">
    <xacro:include filename="robot_core.xacro" />
-   <xacro:include filename="gazebo_control.xacro" />
+   <!-- <xacro:include filename="gazebo_control.xacro" />  -->
    <xacro:include filename="lidar.xacro" />
    <xacro:include filename="camera.xacro" />
-   <!-- <xacro:include filename="ros2_control.xacro"/> -->
+   <xacro:include filename="ros2_control.xacro"/>
 </robot>
